File: Christmas_2022_PCB.kicad_pcb (KiCad board)
At the start: 2 copper layers, 61.4 x 60.5 mm, 45 parts, among them J1 USB_A, J2 SOP8_test_point, J3 SOP8_test_point, SW1 SW_Push, SW2 SW_Push, SW3 SW_SPDT, U1 STM32F030K6Tx, U2 AMS1117-3.3

Commit message: Finished routing. Output gerbers and drill files
Parts:
- moved R1 5.05 mm to (78.0, 77.8), turned to -129 degrees
- moved C3 2.61 mm to (82.2, 75.0)
- moved C2 1.06 mm to (97.6, 75.0)
- moved J1 0.50 mm to (90.0, 113.5)
- moved TH1 0.50 mm to (90.0, 54.5)
- moved C1 0.44 mm to (84.2, 79.5)
- moved D3 0.25 mm to (77.8, 68.2)
- moved D5 0.25 mm to (102.2, 68.2)
- moved R10 0.25 mm to (98.2, 68.2)
- moved R9 0.25 mm to (81.8, 68.2)
- renumbered REF** to TH1
Routing:
- net +3V3: track 69.3 -> 61.8 mm, vias 17 -> 21
- net Net-(R1-Pad1): track 4.12 -> 10.3 mm
- net /LED5: track 15.0 -> 17.9 mm
- net /LED7: track 31.7 -> 32.4 mm
Other:
- board text added: "2022"
- board text added: "Harry Kreicers"
